Commit message: Added transmission & fixed collision geometry

File: manp_description/urdf/manp.xacro (robot description, xacro)
@@ -8,5 +8,5 @@
 	<xacro:property name="base_r" value="1"/>
 	<xacro:property name="base_link_mass" value="1"/>
-	<xacro:property name="link_mass" value="0.01"/>
+	<xacro:property name="link_mass" value="1"/>
 <!-- Links -->
 	<link name="world"/>
@@ -19,4 +19,5 @@
 		</visual>
 		<inertial>
+			<origin xyz="0 0 ${base_h/2}"/>
       			<mass value="${base_link_mass}"/>
       			<inertia
@@ -40,4 +41,5 @@
 		</visual>
 		<inertial>
+			<origin xyz="0 0 ${height/4}"/>
       			<mass value="${link_mass/2}"/>
       			<inertia ixx="${link_mass*height*height/6}" ixy="0.0" ixz="0.0" iyy="${link_mass*height*height/6}" iyz="0.0" izz="1e-10"/>
@@ -58,4 +60,5 @@
 		</visual>
 		<inertial>
+			<origin xyz="0 0 ${height/2}"/>
       			<mass value="${link_mass}"/>
       			<inertia ixx="${link_mass*height*height/3}" ixy="0.0" ixz="0.0" iyy="${link_mass*height*height/3}" iyz="0.0" izz="1e-10"/>
@@ -76,4 +79,5 @@
 		</visual>
 		<inertial>
+			<origin xyz="0 0 ${height/2}"/>
       			<mass value="${link_mass}"/>
       			<inertia ixx="${link_mass*height*height/3}" ixy="0.0" ixz="0.0" iyy="${link_mass*height*height/3}" iyz="0.0" izz="1e-10"/>
@@ -103,5 +107,5 @@
 		<parent link="link1"/>
 		<child link="link2"/>
-		<origin xyz="0 ${-width} ${height/2-0.5}"/>
+		<origin xyz="0 ${-width} ${height/2-0.5}" rpy="0 0 0"/>
 		<axis xyz="0 1 0"/>
 	</joint>
@@ -113,3 +117,45 @@
 	</joint>
 <!-- ###### -->
+<!-- Transmissions -->
+	<transmission name="world_to_base">
+		<type>transmission_interface/SimpleTransmission</type>
+    		<joint name="world_to_base">
+      			<hardwareInterface>EffortJointInterface</hardwareInterface>
+    		</joint>
+    		<actuator name="z-motor">
+      			<mechanicalReduction>1</mechanicalReduction>
+      			<hardwareInterface>EffortJointInterface</hardwareInterface>
+    		</actuator>
+  	</transmission>
+	<transmission name="base_to_link1">
+		<type>transmission_interface/SimpleTransmission</type>
+    		<joint name="base_to_link1">
+      			<hardwareInterface>EffortJointInterface</hardwareInterface>
+    		</joint>
+    		<actuator name="y-motor1">
+      			<mechanicalReduction>1</mechanicalReduction>
+      			<hardwareInterface>EffortJointInterface</hardwareInterface>
+    		</actuator>
+  	</transmission>
+	<transmission name="link1_to_link2">
+		<type>transmission_interface/SimpleTransmission</type>
+    		<joint name="link1_to_link2">
+      			<hardwareInterface>EffortJointInterface</hardwareInterface>
+    		</joint>
+    		<actuator name="y-motor2">
+      			<mechanicalReduction>1</mechanicalReduction>
+      			<hardwareInterface>EffortJointInterface</hardwareInterface>
+    		</actuator>
+  	</transmission>
+	<transmission name="link2_to_link3">
+		<type>transmission_interface/SimpleTransmission</type>
+    		<joint name="link2_to_link3">
+      			<hardwareInterface>EffortJointInterface</hardwareInterface>
+    		</joint>
+    		<actuator name="y-motor3">
+      			<mechanicalReduction>1</mechanicalReduction>
+      			<hardwareInterface>EffortJointInterface</hardwareInterface>
+    		</actuator>
+  	</transmission>
+<!-- ############# -->
 </robot>

Commit message: Removed unneeded transmission

File: manp_description/urdf/manp.xacro (robot description, xacro)
@@ -128,14 +128,4 @@
     		</actuator>
   	</transmission>
-	<transmission name="base_to_link1">
-		<type>transmission_interface/SimpleTransmission</type>
-    		<joint name="base_to_link1">
-      			<hardwareInterface>EffortJointInterface</hardwareInterface>
-    		</joint>
-    		<actuator name="y-motor1">
-      			<mechanicalReduction>1</mechanicalReduction>
-      			<hardwareInterface>EffortJointInterface</hardwareInterface>
-    		</actuator>
-  	</transmission>
 	<transmission name="link1_to_link2">
 		<type>transmission_interface/SimpleTransmission</type>

Commit message: Rewrited node for control, changed joint base_to_link1 to prismatic with zero limits. Still collapses when moved

File: manp_description/urdf/manp.xacro (robot description, xacro)
@@ -98,9 +98,9 @@
 		<axis xyz="0 0 1"/>
 	</joint>
-	<joint name="base_to_link1" type="fixed">
+	<joint name="base_to_link1" type="prismatic">
 		<parent link="base_link"/>
 		<child link="link1"/>
 		<origin xyz="0 0 ${base_h}"/>
-		<axis xyz="0 1 0"/>
+		<limit effort="1" lower="0.0" upper="0.0" velocity="1"/>
 	</joint>
 	<joint name="link1_to_link2" type="continuous">

Commit message: Hunting for bugs. Still not found

File: manp_description/urdf/manp.xacro (robot description, xacro)
@@ -7,6 +7,6 @@
 	<xacro:property name="base_h" value="0.5"/>
 	<xacro:property name="base_r" value="1"/>
-	<xacro:property name="base_link_mass" value="1"/>
-	<xacro:property name="link_mass" value="1"/>
+	<xacro:property name="base_link_mass" value="20"/>
+	<xacro:property name="link_mass" value="40"/>
 <!-- Links -->
 	<link name="world"/>
@@ -107,5 +107,5 @@
 		<parent link="link1"/>
 		<child link="link2"/>
-		<origin xyz="0 ${-width} ${height/2-0.5}" rpy="0 0 0"/>
+		<origin xyz="0 ${-(width+1)} ${height/2-0.5}" rpy="0 0 0"/>
 		<axis xyz="0 1 0"/>
 	</joint>
@@ -113,5 +113,5 @@
 		<parent link="link2"/>
 		<child link="link3"/>
-		<origin xyz="0 ${width} ${height-0.5}"/>
+		<origin xyz="0 ${width+1} ${height-0.5}"/>
 		<axis xyz="0 1 0"/>
 	</joint>

Commit message: Fixed the bug with all links jumping to world origins

File: manp_description/urdf/manp.xacro (robot description, xacro)
@@ -22,6 +22,6 @@
       			<mass value="${base_link_mass}"/>
       			<inertia
-				ixx="${base_link_mass*(3*base_r*base_r+base_h*base_h)/12}" ixy="0.0" ixz="0.0"
-				iyy="${base_link_mass*(3*base_r*base_r+base_h*base_h)/12}" iyz="0.0" izz="${base_link_mass*base_r*base_r/2}"
+				ixx="${base_link_mass*(3*base_r*base_r+base_h*base_h)/12}" ixy="1e-3" ixz="1e-3"
+				iyy="${base_link_mass*(3*base_r*base_r+base_h*base_h)/12}" iyz="1e-3" izz="${base_link_mass*base_r*base_r/2}"
 			/>
     		</inertial>
@@ -43,5 +43,5 @@
 			<origin xyz="0 0 ${height/4}"/>
       			<mass value="${link_mass/2}"/>
-      			<inertia ixx="${link_mass*height*height/6}" ixy="0.0" ixz="0.0" iyy="${link_mass*height*height/6}" iyz="0.0" izz="1e-10"/>
+      			<inertia ixx="${link_mass*height*height/6}" ixy="1e-3" ixz="1e-3" iyy="${link_mass*height*height/6}" iyz="1e-3" izz="1e-3"/>
     		</inertial>
 		<collision>
@@ -62,5 +62,5 @@
 			<origin xyz="0 0 ${height/2}"/>
       			<mass value="${link_mass}"/>
-      			<inertia ixx="${link_mass*height*height/3}" ixy="0.0" ixz="0.0" iyy="${link_mass*height*height/3}" iyz="0.0" izz="1e-10"/>
+      			<inertia ixx="${link_mass*height*height/3}" ixy="1e-3" ixz="1e-3" iyy="${link_mass*height*height/3}" iyz="1e-3" izz="1e-3"/>
     		</inertial>
 		<collision>
@@ -81,5 +81,5 @@
 			<origin xyz="0 0 ${height/2}"/>
       			<mass value="${link_mass}"/>
-      			<inertia ixx="${link_mass*height*height/3}" ixy="0.0" ixz="0.0" iyy="${link_mass*height*height/3}" iyz="0.0" izz="1e-10"/>
+      			<inertia ixx="${link_mass*height*height/3}" ixy="1e-3" ixz="1e-3" iyy="${link_mass*height*height/3}" iyz="1e-3" izz="1e-3"/>
     		</inertial>
 		<collision>

Commit message: Fixed models spacing in joints to normal & added self colision to every joint

File: manp_description/urdf/manp.xacro (robot description, xacro)
@@ -98,14 +98,13 @@
 		<axis xyz="0 0 1"/>
 	</joint>
-	<joint name="base_to_link1" type="prismatic">
+	<joint name="base_to_link1" type="fixed">
 		<parent link="base_link"/>
 		<child link="link1"/>
 		<origin xyz="0 0 ${base_h}"/>
-		<limit effort="1" lower="0.0" upper="0.0" velocity="1"/>
 	</joint>
 	<joint name="link1_to_link2" type="continuous">
 		<parent link="link1"/>
 		<child link="link2"/>
-		<origin xyz="0 ${-(width+1)} ${height/2-0.5}" rpy="0 0 0"/>
+		<origin xyz="0 ${-width-0.1} ${height/2-0.5}" rpy="0 0 0"/>
 		<axis xyz="0 1 0"/>
 	</joint>
@@ -113,5 +112,5 @@
 		<parent link="link2"/>
 		<child link="link3"/>
-		<origin xyz="0 ${width+1} ${height-0.5}"/>
+		<origin xyz="0 ${width+0.1} ${height-0.5}"/>
 		<axis xyz="0 1 0"/>
 	</joint>
@@ -149,4 +148,18 @@
   	</transmission>
 <!-- ############# -->
+<!-- Setting self collide for every link -->
+	<gazebo reference="base_link">
+    		<selfCollide>true</selfCollide>
+	</gazebo>
+	<gazebo reference="link1">
+    		<selfCollide>true</selfCollide>
+	</gazebo>
+	<gazebo reference="link2">
+    		<selfCollide>true</selfCollide>
+	</gazebo>
+	<gazebo reference="link3">
+    		<selfCollide>true</selfCollide>
+	</gazebo>
+<!-- ################################# -->
 	<gazebo>
     		<plugin name="gazebo_ros_control" filename="libgazebo_ros_control.so">

Commit message: Final fixes to model

File: manp_description/urdf/manp.xacro (robot description, xacro)
@@ -106,5 +106,5 @@
 		<parent link="link1"/>
 		<child link="link2"/>
-		<origin xyz="0 ${-width-0.1} ${height/2-0.5}" rpy="0 0 0"/>
+		<origin xyz="0 ${-width} ${height/2-0.5}" rpy="0 0 0"/>
 		<axis xyz="0 1 0"/>
 	</joint>
@@ -112,5 +112,5 @@
 		<parent link="link2"/>
 		<child link="link3"/>
-		<origin xyz="0 ${width+0.1} ${height-0.5}"/>
+		<origin xyz="0 ${width} ${height-0.5}"/>
 		<axis xyz="0 1 0"/>
 	</joint>
@@ -154,10 +154,16 @@
 	<gazebo reference="link1">
     		<selfCollide>true</selfCollide>
+		<mu1>0.2</mu1>
+   		<mu2>0.2</mu2>
 	</gazebo>
 	<gazebo reference="link2">
     		<selfCollide>true</selfCollide>
+		<mu1>0.2</mu1>
+    		<mu2>0.2</mu2>
 	</gazebo>
 	<gazebo reference="link3">
     		<selfCollide>true</selfCollide>
+		<mu1>0.2</mu1>
+    		<mu2>0.2</mu2>
 	</gazebo>
 <!-- ################################# -->

Commit message: Added friction to the joints

File: manp_description/urdf/manp.xacro (robot description, xacro)
@@ -108,4 +108,5 @@
 		<origin xyz="0 ${-width} ${height/2-0.5}" rpy="0 0 0"/>
 		<axis xyz="0 1 0"/>
+		<!-- <limit lower="0" upper="${pi}" effort="10000" velocity="1"/> -->
 	</joint>
 	<joint name="link2_to_link3" type="continuous">

Commit message: Still hunting for goddamn bugs. One function only checked

File: manp_description/urdf/manp.xacro (robot description, xacro)
@@ -92,9 +92,9 @@
 <!-- ########### -->
 <!-- Joints -->
-	<joint name="world_to_base" type="continuous">
+	<joint name="world_to_base" type="fixed">
 		<parent link="world"/>
 		<child link="base_link"/>
 		<origin xyz="0 0 0"/>
-		<axis xyz="0 0 1"/>
+		<!-- <axis xyz="0 0 1"/>-->
 	</joint>
 	<joint name="base_to_link1" type="fixed">
@@ -113,10 +113,10 @@
 		<parent link="link2"/>
 		<child link="link3"/>
-		<origin xyz="0 ${width} ${height-0.5}"/>
+		<origin xyz="0 ${width} ${height-0.5}" rpy="0 1 0"/>
 		<axis xyz="0 1 0"/>
 	</joint>
 <!-- ###### -->
 <!-- Transmissions -->
-	<transmission name="world_to_base">
+	<!--<transmission name="world_to_base">
 		<type>transmission_interface/SimpleTransmission</type>
     		<joint name="world_to_base">
@@ -127,5 +127,5 @@
       			<hardwareInterface>EffortJointInterface</hardwareInterface>
     		</actuator>
-  	</transmission>
+  	</transmission> -->
 	<transmission name="link1_to_link2">
 		<type>transmission_interface/SimpleTransmission</type>
@@ -155,16 +155,10 @@
 	<gazebo reference="link1">
     		<selfCollide>true</selfCollide>
-		<mu1>0.2</mu1>
-   		<mu2>0.2</mu2>
 	</gazebo>
 	<gazebo reference="link2">
     		<selfCollide>true</selfCollide>
-		<mu1>0.2</mu1>
-    		<mu2>0.2</mu2>
 	</gazebo>
 	<gazebo reference="link3">
     		<selfCollide>true</selfCollide>
-		<mu1>0.2</mu1>
-    		<mu2>0.2</mu2>
 	</gazebo>
 <!-- ################################# -->

Commit message: Bugs slaughtered. All working fine

File: manp_description/urdf/manp.xacro (robot description, xacro)
@@ -3,10 +3,10 @@
 <!-- Constants -->
 	<xacro:property name="pi" value="3.14159265359"/>
-	<xacro:property name="width" value="0.5"/>
-	<xacro:property name="height" value="4"/>
-	<xacro:property name="base_h" value="0.5"/>
-	<xacro:property name="base_r" value="1"/>
-	<xacro:property name="base_link_mass" value="20"/>
-	<xacro:property name="link_mass" value="40"/>
+	<xacro:property name="width" value="0.05"/>
+	<xacro:property name="height" value="0.4"/>
+	<xacro:property name="base_h" value="0.05"/>
+	<xacro:property name="base_r" value="0.1"/>
+	<xacro:property name="base_link_mass" value="2"/>
+	<xacro:property name="link_mass" value="4"/>
 <!-- Links -->
 	<link name="world"/>
@@ -92,9 +92,10 @@
 <!-- ########### -->
 <!-- Joints -->
-	<joint name="world_to_base" type="fixed">
+	<joint name="world_to_base" type="continuous">
 		<parent link="world"/>
 		<child link="base_link"/>
 		<origin xyz="0 0 0"/>
-		<!-- <axis xyz="0 0 1"/>-->
+		<axis xyz="0 0 1"/>
+		<limit lower="${-pi/2}" upper="${pi/2}" effort="10000" velocity="1"/>
 	</joint>
 	<joint name="base_to_link1" type="fixed">
@@ -103,20 +104,21 @@
 		<origin xyz="0 0 ${base_h}"/>
 	</joint>
-	<joint name="link1_to_link2" type="continuous">
+	<joint name="link1_to_link2" type="revolute">
 		<parent link="link1"/>
 		<child link="link2"/>
-		<origin xyz="0 ${-width} ${height/2-0.5}" rpy="0 0 0"/>
+		<origin xyz="0 ${-width} ${height/2}" rpy="0 0 0"/>
 		<axis xyz="0 1 0"/>
-		<!-- <limit lower="0" upper="${pi}" effort="10000" velocity="1"/> -->
+		<limit lower="${-pi/2}" upper="${pi/2}" effort="10000" velocity="1"/>
 	</joint>
-	<joint name="link2_to_link3" type="continuous">
+	<joint name="link2_to_link3" type="revolute">
 		<parent link="link2"/>
 		<child link="link3"/>
-		<origin xyz="0 ${width} ${height-0.5}" rpy="0 1 0"/>
+		<origin xyz="0 ${width} ${height}" rpy="0 1 0"/>
 		<axis xyz="0 1 0"/>
+		<limit lower="${-pi/2}" upper="${pi/2}" effort="10000" velocity="1"/>
 	</joint>
 <!-- ###### -->
 <!-- Transmissions -->
-	<!--<transmission name="world_to_base">
+	<transmission name="world_to_base">
 		<type>transmission_interface/SimpleTransmission</type>
     		<joint name="world_to_base">
@@ -127,5 +129,5 @@
       			<hardwareInterface>EffortJointInterface</hardwareInterface>
     		</actuator>
-  	</transmission> -->
+  	</transmission>
 	<transmission name="link1_to_link2">
 		<type>transmission_interface/SimpleTransmission</type>
@@ -151,10 +153,13 @@
 <!-- Setting self collide for every link -->
 	<gazebo reference="base_link">
+		<gravity>0</gravity>
     		<selfCollide>true</selfCollide>
 	</gazebo>
 	<gazebo reference="link1">
+		<gravity>0</gravity>
     		<selfCollide>true</selfCollide>
 	</gazebo>
 	<gazebo reference="link2">
+		<gravity>0</gravity>
     		<selfCollide>true</selfCollide>
 	</gazebo>
